File: board/schematic.sch (EAGLE design)
At the start: 53 parts, among them J2 AVR_SPI_PROG_3X2PTH, U1 328P, U2 SN74HC595N, U3 SN74HC595N, U4 SN74HC595N, U5 SN74HC595N

Commit message: Fix crossed rx/tx
Connections:
- net RXD: now also J1.TXO; no longer J1.RXI
- net TXD: now also J1.RXI; no longer J1.TXO
Changed lines of the file:
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@@
 </segment>
 <segment>
-<pinref part="J1" gate="G$1" pin="RXI"/>
-<wire x1="78.74" y1="38.1" x2="73.66" y2="38.1" width="0.1524" layer="91"/>
-<label x="68.58" y="38.1" size="1.778" layer="95"/>
+<pinref part="J1" gate="G$1" pin="TXO"/>
+<wire x1="78.74" y1="35.56" x2="73.66" y2="35.56" width="0.1524" layer="91"/>
+<label x="68.58" y="35.56" size="1.778" layer="95"/>
 </segment>
 </net>
@@
 </segment>
 <segment>
-<pinref part="J1" gate="G$1" pin="TXO"/>
-<wire x1="78.74" y1="35.56" x2="73.66" y2="35.56" width="0.1524" layer="91"/>
-<label x="68.58" y="35.56" size="1.778" layer="95"/>
+<pinref part="J1" gate="G$1" pin="RXI"/>
+<wire x1="78.74" y1="38.1" x2="73.66" y2="38.1" width="0.1524" layer="91"/>
+<label x="68.58" y="38.1" size="1.778" layer="95"/>
 </segment>
 </net>
